File: EMG_hand_sensor/EMG_hand_sensor.kicad_pcb (KiCad board)
At the start: 4 copper layers, 78 x 41.5 mm, 50 parts, among them J1 USB_C_Receptacle_USB2.0_16P, J2 Conn_01x04_Pin, J4 AudioJack3, J5 AudioJack3, J6 AudioJack3, SW1 SW_SPDT, U1 USBLC6-2SC6, U2 STM32F103C8Tx, U3 INA128, U5 INA128, U7 LT1762, U9 INA128, Y1 16MHz

Commit message: done with most of the routing
Parts:
- removed R10, R5, R6: 50R, Resistor_SMD:R_0805_2012Metric_Pad1.20x1.40mm_HandSolder
- added C18: 100nF, Capacitor_SMD:C_0805_2012Metric_Pad1.18x1.45mm_HandSolder, F.Cu at (196.5, 60.4)
- added C20: 100nF, Capacitor_SMD:C_0805_2012Metric_Pad1.18x1.45mm_HandSolder, F.Cu at (195.8, 86.7)
- added C21: 100nF, Capacitor_SMD:C_0805_2012Metric_Pad1.18x1.45mm_HandSolder, F.Cu at (196.6, 62.8)
- added RV1: 500R, Potentiometer_SMD:Potentiometer_Bourns_3214W_Vertical, F.Cu at (189.9, 55.5)
- added RV2: 500R, Potentiometer_SMD:Potentiometer_Bourns_3214W_Vertical, F.Cu at (194.2, 72.7)
- added RV3: 500R, Potentiometer_SMD:Potentiometer_Bourns_3214W_Vertical, F.Cu at (189.5, 86.5)
- moved C7 27.6 mm to (162.1, 80.2), turned to -90 degrees
- moved C8 23.5 mm to (164.3, 80.2), turned to -90 degrees
- moved R9 2.77 mm to (155.0, 78.2)
- moved R12 2.17 mm to (187.9, 74.5), turned to 180 degrees
- moved C17 1.89 mm to (192.0, 76.5)
- moved Y1 1.61 mm to (183.6, 78.4)
- moved H1 1.24 mm to (147.6, 86.7)
- moved U1 1.16 mm to (163.2, 73.0)
- moved H2 0.96 mm to (147.3, 54.2)
Connections:
- U2 pad 10: /O1 -> unconnected-(U2-PA0-Pad10)
- U9 pad 1: Net-(R10-Pad1) -> /RV3_1
- U9 pad 8: Net-(R10-Pad2) -> /RV3_3
Routing:
- net GND: track 0.44 -> 118.0 mm, vias 0 -> 59
- net +3.3V: track 0.00 -> 80.5 mm, vias 0 -> 26
- net /RV3_1: track 0.00 -> 49.5 mm
- net +1V6: track 0.00 -> 32.4 mm, vias 0 -> 4
- net /O4: track 0.00 -> 22.4 mm
- net VBUS: track 0.00 -> 21.5 mm, vias 0 -> 4
- net /O2: track 0.00 -> 19.8 mm
- net /E1: track 0.00 -> 19.0 mm
- net /E5: track 0.42 -> 19.1 mm
- net Net-(RV1-Pad1): track 0.00 -> 18.5 mm
- net /E8: track 0.00 -> 17.5 mm
- net /HSE_IN: track 0.00 -> 12.4 mm
- net /RV3_3: track 0.00 -> 10.9 mm
- net /O3: track 0.00 -> 10.8 mm
- net Net-(RV1-Pad3): track 0.00 -> 10.7 mm
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Other:
- board size 78 x 41.5 mm -> 71.4 x 41.5 mm
