File: EMG_hand_sensor/EMG_hand_sensor.kicad_pcb (KiCad board)
At the start: 4 copper layers, 71.4 x 41.5 mm, 53 parts, among them J1 USB_C_Receptacle_USB2.0_16P, J2 Conn_01x04_Pin, J4 AudioJack3, J5 AudioJack3, J6 AudioJack3, SW1 SW_SPDT, U1 USBLC6-2SC6, U2 STM32F103C8Tx, U3 INA128, U5 INA128, U7 LT1762, U9 INA128, Y1 16MHz

Commit message: Finalising board running DRC
Parts:
- moved FID2 0.56 mm to (198.0, 89.2)
Routing:
- net GND: track 118.0 -> 308.2 mm
- net +3.3V: track 80.5 -> 142.3 mm
- net +3.3VA: track 6.02 -> 32.5 mm, vias 3 -> 4
- net /USB_D-: track 0.00 -> 21.5 mm
- net /USB_D+: track 0.00 -> 21.5 mm
- net +1V6: track 32.4 -> 53.0 mm
- net VBUS: track 21.5 -> 36.5 mm, vias 4 -> 3
- net /NRST: track 0.00 -> 5.01 mm
- net /O2: track 19.8 -> 23.5 mm

Commit message: done DRC final checks
Routing:
- net +3.3V: track 142.3 -> 83.3 mm
- net GND: track 308.2 -> 271.5 mm, vias 59 -> 66
- net /USB_D-: track 21.5 -> 26.1 mm
- net /USB_D+: track 21.5 -> 26.1 mm
- net +3.3VA: track 32.5 -> 35.5 mm
- net /CC2: track 5.69 -> 4.40 mm
- net VBUS: track 36.5 -> 37.5 mm, vias 3 -> 2
- added copper zone on B.Cu, net +3.3V
Other:
- outline, holes or cut-outs redrawn

Commit message: ready for ordering
Parts:
- moved D1 0.06 mm to (156.5, 86.8)
Routing:
- net +3.3VA: track 35.5 -> 34.9 mm
Other:
- board size 71.4 x 41.5 mm -> 73.9 x 41.5 mm
Changed lines of the file:
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@@
 		(tags "fiducial")
 		(property "Reference" "FID2"
-			(at 0 -1.95 0)
+			(at -3 0.25 0)
 			(layer "F.SilkS")
 			(effects
@@
 		(tags "capacitor handsolder")
 		(property "Reference" "C7"
-			(at 0 -1.68 90)
+			(at 0 1.84 90)
 			(layer "F.SilkS")
 			(effects
@@
 		(tags "LQFP QFP CASE-932AA CASE-932-03 C48-1 C48-2 C48-3 C48-5 C48-6 C48-6C PT0048A")
 		(property "Reference" "U2"
-			(at 0 -5.85 0)
+			(at 0 0 0)
 			(layer "F.SilkS")
 			(effects
@@
 		(tags "capacitor handsolder")
 		(property "Reference" "C18"
-			(at 0 -1.68 0)
+			(at 3.4525 0.14 0)
 			(layer "F.SilkS")
 			(effects
@@
 		(tags "resistor handsolder")
 		(property "Reference" "R11"
-			(at 0 -1.65 0)
+			(at 0 1.5 0)
 			(layer "F.SilkS")
 			(effects
@@
 		(tags "capacitor handsolder")
 		(property "Reference" "C8"
-			(at 0 -1.68 90)
+			(at 0.055 -1.66 90)
 			(layer "F.SilkS")
 			(effects
@@
 		(tags "capacitor handsolder")
 		(property "Reference" "C4"
-			(at 0 0 90)
+			(at 3 0 180)
 			(layer "F.SilkS")
 			(effects
@@
 		(tags "capacitor handsolder")
 		(property "Reference" "C6"
-			(at 0 -1.68 90)
+			(at 2.7125 0 180)
 			(layer "F.SilkS")
 			(effects
@@
 		(tags "resistor handsolder")
 		(property "Reference" "R3"
-			(at 0 -1.65 90)
+			(at 0 -2.5 90)
 			(layer "F.SilkS")
 			(effects
@@
 		(tags "3.5mm audio cui horizontal jack stereo")
 		(property "Reference" "J5"
-			(at 0 -9.9 90)
+			(at 0 0 90)
 			(layer "F.SilkS")
 			(effects
@@
 		(tags "capacitor handsolder")
 		(property "Reference" "C15"
-			(at 0 -1.68 0)
+			(at 0 2 0)
 			(layer "F.SilkS")
 			(effects
@@
 	(footprint "Diode_SMD:D_0805_2012Metric"
 		(layer "F.Cu")
-		(at 156.5625 86.75)
+		(at 156.5 86.75)
 		(descr "Diode SMD 0805 (2012 Metric), square (rectangular) end terminal, IPC-7351 nominal, (Body size source: https://docs.google.com/spreadsheets/d/1BsfQQcO9C6DZCsRaXUlFlo91Tg2WpOkGARC1WS5S8t0/edit?usp=sharing), generated with kicad-footprint-generator")
 		(tags "diode")
 		(property "Reference" "D1"
-			(at 0 -1.65 0)
+			(at 0 1.75 0)
 			(layer "F.SilkS")
 			(effects
@@
 		(tags "resistor handsolder")
 		(property "Reference" "R1"
-			(at 0 -1.65 0)
+			(at 0 0 0)
 			(layer "F.SilkS")
 			(effects
@@
 		(tags "capacitor handsolder")
 		(property "Reference" "C3"
-			(at 0 0 90)
+			(at 3.0375 0 180)
 			(layer "F.SilkS")
 			(effects
@@
 		(tags "capacitor handsolder")
 		(property "Reference" "C1"
-			(at -3.9175 -1.48 90)
+			(at 0 1.75 90)
 			(layer "F.SilkS")
 			(effects
@@
 		(tags "capacitor handsolder")
 		(property "Reference" "C11"
-			(at 0 -1.68 0)
+			(at 0 1.75 0)
 			(layer "F.SilkS")
 			(effects
@@
 		(tags "Potentiometer vertical Bourns 3214W")
 		(property "Reference" "RV2"
-			(at 0 -3.5 0)
+			(at 4.06 -0.21 0)
 			(layer "F.SilkS")
 			(effects
@@
 		(tags "fiducial")
 		(property "Reference" "FID3"
-			(at 0 -1.95 0)
+			(at 1.5 2 0)
 			(layer "F.SilkS")
 			(effects
@@
 		(tags "capacitor handsolder")
 		(property "Reference" "C12"
-			(at 0 -1.68 90)
+			(at 0.5 -1.75 90)
 			(layer "F.SilkS")
 			(effects
@@
 		(descr "SMD3225/4, Crystal, 3.2x2.5mm package, SMD, generated with kicad-footprint-generator make_crystal.py, http://www.txccrystal.com/images/pdf/7m-accuracy.pdf")
 		(property "Reference" "Y1"
-			(at 0 -2.45 0)
+			(at 0 2.61 0)
 			(layer "F.SilkS")
 			(effects
@@
 		(tags "capacitor handsolder")
 		(property "Reference" "C2"
-			(at 0 -1.68 90)
+			(at 3 0 0)
 			(layer "F.SilkS")
 			(effects
@@
 		(tags "Potentiometer vertical Bourns 3214W")
 		(property "Reference" "RV1"
-			(at 0 -3.5 0)
+			(at 0 0 0)
 			(layer "F.SilkS")
 			(effects
@@
 		(tags "capacitor handsolder")
 		(property "Reference" "C21"
-			(at 0 -1.68 0)
+			(at 3.44 -0.03 0)
 			(layer "F.SilkS")
 			(effects
@@
 		(tags "capacitor handsolder")
 		(property "Reference" "C5"
-			(at 0 0 90)
+			(at 3 0 180)
 			(layer "F.SilkS")
 			(effects
@@
 		(tags "resistor handsolder")
 		(property "Reference" "R8"
-			(at -11.5 -2.65 0)
+			(at 0 0 0)
 			(layer "F.SilkS")
 			(effects
@@
 		(tags "capacitor handsolder")
 		(property "Reference" "C9"
-			(at 0 -1.68 90)
+			(at 0 1.817621 90)
 			(layer "F.SilkS")
 			(effects
@@
 		(tags "Potentiometer vertical Bourns 3214W")
 		(property "Reference" "RV3"
-			(at 0 -3.5 0)
+			(at 0 -0.05 0)
 			(layer "F.SilkS")
 			(effects
@@
 		(tags "MSOP SO")
 		(property "Reference" "U7"
-			(at 0 -2.45 90)
+			(at -0.25 -0.067621 90)
 			(layer "F.SilkS")
 			(effects
@@
 		(tags "3.5mm audio cui horizontal jack stereo")
 		(property "Reference" "J6"
-			(at 0 -9.9 90)
+			(at 0 0 90)
 			(layer "F.SilkS")
 			(effects
@@
 		(tags "3.5mm audio cui horizontal jack stereo")
 		(property "Reference" "J4"
-			(at 0 -9.9 90)
+			(at 0 0 90)
 			(layer "F.SilkS")
 			(effects
@@
 		(tags "capacitor handsolder")
 		(property "Reference" "C14"
-			(at 0 -1.68 90)
+			(at 0 -2.5 90)
 			(layer "F.SilkS")
 			(effects
@@
 		(tags "capacitor handsolder")
 		(property "Reference" "C17"
-			(at 0 -1.68 0)
+			(at 3.96 0.3 0)
 			(layer "F.SilkS")
 			(effects
@@
 		(tags "resistor handsolder")
 		(property "Reference" "R14"
-			(at 0 -1.65 90)
+			(at 0 2 270)
 			(layer "F.SilkS")
 			(effects
@@
 		(tags "capacitor handsolder")
 		(property "Reference" "C20"
-			(at 0 -1.68 0)
+			(at 0 0 0)
 			(layer "F.SilkS")
 			(effects
@@
 	)
 	(gr_line
-		(start 178 91.25)
-		(end 143.840002 91.494)
+		(start 217.75 50)
+		(end 217.75 91)
 		(stroke
 			(width 0.05)
@@
 	(gr_line
 		(start 178 91.25)
-		(end 215.19 90.97)
+		(end 143.840002 91.494)
 		(stroke
 			(width 0.05)
@@
 	)
 	(gr_line
-		(start 215.21 50)
+		(start 178 91.25)
 		(end 215.19 90.97)
 		(stroke
@@
 		(layer "Edge.Cuts")
 	)
+	(gr_line
+		(start 215.21 50)
+		(end 217.75 50)
+		(stroke
+			(width 0.05)
+			(type default)
+		)
+		(layer "Edge.Cuts")
+	)
+	(gr_line
+		(start 217.75 91)
+		(end 215.19 90.97)
+		(stroke
+			(width 0.05)
+			(type default)
+		)
+		(layer "Edge.Cuts")
+	)
 	(segment
 		(start 170.75 70.25)
@@
 	)
 	(segment
-		(start 182.1625 71.25)
-		(end 183.75 71.25)
-		(width 0.3)
-		(layer "F.Cu")
-		(net 1)
-	)
-	(segment
 		(start 162.09 79.195)
 		(end 162.09 77.98)
@@
 	)
 	(segment
+		(start 182.1625 71.25)
+		(end 183.5 71.25)
+		(width 0.3)
+		(layer "F.Cu")
+		(net 1)
+	)
+	(segment
 		(start 164.34 77.98)
 		(end 164.32 77.96)
@@
 	)
 	(via
-		(at 183.75 71.25)
+		(at 183.5 71.25)
 		(size 0.7)
 		(drill 0.3)
@@
 	)
 	(segment
-		(start 170.571 69.169)
+		(start 183.5 71)
 		(end 181.669 69.169)
 		(width 0.5)
@@
 	(segment
 		(start 183.5 71.25)
-		(end 183.75 71.25)
-		(width 0.5)
-		(layer "B.Cu")
-		(net 1)
-	)
-	(segment
-		(start 169.37 70.37)
-		(end 169.45 70.29)
-		(width 0.5)
-		(layer "B.Cu")
-		(net 1)
-	)
-	(segment
-		(start 169.45 70.29)
-		(end 170.571 69.169)
+		(end 183.5 71)
 		(width 0.5)
 		(layer "B.Cu")
@@
 	)
 	(segment
-		(start 181.669 69.169)
-		(end 183.75 71.25)
+		(start 164.32 77.96)
+		(end 164.31 77.95)
 		(width 0.5)
 		(layer "B.Cu")
@@
 	)
 	(segment
-		(start 164.32 77.96)
-		(end 164.31 77.95)
+		(start 181.669 69.169)
+		(end 170.571 69.169)
 		(width 0.5)
 		(layer "B.Cu")
@@
 	)
 	(segment
+		(start 170.571 69.169)
+		(end 169.37 70.37)
+		(width 0.5)
+		(layer "B.Cu")
+		(net 1)
+	)
+	(segment
 		(start 170.96 54.58875)
 		(end 170.96 55.79125)
@@
 	)
 	(segment
+		(start 180.75 76.6625)
+		(end 180.75 79)
+		(width 0.3)
+		(layer "F.Cu")
+		(net 14)
+	)
+	(segment
 		(start 164.72 66.2)
 		(end 164.72 64.99)
@@
 	)
 	(segment
+		(start 180.75 79)
+		(end 180.5 79.25)
+		(width 0.3)
+		(layer "F.Cu")
+		(net 14)
+	)
+	(segment
 		(start 175.25 68.3375)
 		(end 175.25 66.28)
@@
 	)
 	(segment
+		(start 180.5 79.25)
+		(end 180.5 84.25)
+		(width 0.3)
+		(layer "F.Cu")
+		(net 14)
+	)
+	(segment
 		(start 158.54 86.8)
 		(end 157.33 86.8)
@@
 		(layer "F.Cu")
 		(net 14)
-	)
-	(segment
-		(start 180.75 76.6625)
-		(end 180.75 84)
-		(width 0.3)
-		(layer "F.Cu")
-		(net 14)
